Commit message: update project to work with tug setup

File: robotino_description/urdf/robotino_body.xacro (robot description, xacro)
@@ -51,5 +51,5 @@
     <laser name="laser" parent="base_link">
       <!--origin xyz="-0.022 0 0.232" rpy="0 0 0"/-->
-      <origin xyz="0.1 0 0" rpy="0 0 0"/>
+      <origin xyz="0.12 0 0" rpy="0 0 0"/>
     </laser>
     <!--laser name="laser" parent="base_link"-->
