Commit message: changed urdf to fit robot
fixed xacro definitions

File: robotino_description/urdf/robotino.urdf (robot description, URDF)
Before this commit: robot robotino, 8 links, 7 joints
Joints:
- joint laser_joint: origin xyz=-0.022 10 0.232 rpy=0 0 0 -> xyz=0.0 0  0.232 rpy=0 0 0

File: robotino_description/urdf/robotino.urdf.xacro (robot description, xacro)
@@ -1,7 +1,7 @@
 <?xml version="1.0"?>
-<robot name="robotino">
+<robot xmlns:xacro="http://www.ros.org/wiki/xacro" name="robotino">
   <!-- Include files -->
-  <include filename="$(find robotino_description)/urdf/robotino_body.xacro"/>
-  <include filename="$(find robotino_description)/urdf/robotino_hardware.xacro"/>
-  <robotino_body />
+    <xacro:include filename="$(find robotino_description)/urdf/robotino_hardware.xacro"/>
+    <xacro:include filename="$(find robotino_description)/urdf/robotino_body.xacro"/>
+   <robotino_body />
 </robot>

File: robotino_description/urdf/robotino_body.xacro (robot description, xacro)
@@ -1,10 +1,10 @@
 <?xml version="1.0"?>
-<robot>
-  <property name="M_PI" value="3.14159"/>
-  <property name="M_SCALE" value="0.01"/>
-  <property name="BASE_RADIUS" value="0.18"/>
-  <property name="BASE_HEIGHT" value="0.05"/>
-  <property name="BASE_MASS" value="20"/>
-  <macro name="robotino_body">
+<robot xmlns:xacro="http://www.ros.org/wiki/xacro">
+  <xacro:property name="M_PI" value="3.14159"/>
+  <xacro:property name="M_SCALE" value="0.01"/>
+  <xacro:property name="BASE_RADIUS" value="0.18"/>
+  <xacro:property name="BASE_HEIGHT" value="0.05"/>
+  <xacro:property name="BASE_MASS" value="20"/>
+  <xacro:macro name="robotino_body">
   	<link name="base_link">
       <inertial>
@@ -28,32 +28,29 @@
       </collision>
     </link>
-    <wheel name="wheel0" parent="base_link">
+    <xacro:wheel name="wheel0" parent="base_link">
       <origin xyz="0.065 0.11 0.04" rpy="0 0 ${M_PI/3}"/>
       <axis xyz="-1 0 0"/>
-    </wheel>
-    <wheel name="wheel1" parent="base_link">
+    </xacro:wheel>
+    <xacro:wheel name="wheel1" parent="base_link">
       <origin xyz="-0.13 0 0.04" rpy="0 0 0"/>
       <axis xyz="1 0 0"/>
-    </wheel>
-    <wheel name="wheel2" parent="base_link">
+    </xacro:wheel>
+    <xacro:wheel name="wheel2" parent="base_link">
       <origin xyz="0.065 -0.11 0.04" rpy="0 0 -${M_PI/3}"/>
       <axis xyz="-1 0 0"/>
-    </wheel>
-    <command_bridge name="command_bridge" parent="base_link">
+    </xacro:wheel>
+    <xacro:command_bridge name="command_bridge" parent="base_link">
       <origin xyz="-0.05 0 0.13" rpy="0 0 ${M_PI/2}"/>
-    </command_bridge>
-    <camera name="camera" parent="base_link">
+    </xacro:command_bridge>
+    <xacro:camera name="camera" parent="base_link">
       <origin xyz="0.044 0 0.07" rpy="0 0 ${M_PI/2}"/>
-    </camera>
-    <anglebracketusb name="anglebracketusb" parent="base_link">
+    </xacro:camera>
+    <xacro:anglebracketusb name="anglebracketusb" parent="base_link">
       <origin xyz="0.008 0 0.137" rpy="0 0 ${M_PI/2}"/>
-    </anglebracketusb>
-    <laser name="laser" parent="base_link">
+    </xacro:anglebracketusb>
+    <xacro:laser name="laser" parent="base_link">
       <!--origin xyz="-0.022 0 0.232" rpy="0 0 0"/-->
-      <origin xyz="0.12 0 0" rpy="0 0 0"/>
-    </laser>
-    <!--laser name="laser" parent="base_link"-->
-      <!--origin xyz="0.12 0 ${BASE_HEIGHT/2}" rpy="0 0 0"/-->
-    <!--/laser-->
-  </macro>
+      <origin xyz="0.0 0  0.232" rpy="0 0 0"/>
+    </xacro:laser>
+  </xacro:macro>
 </robot>

File: robotino_description/urdf/robotino_hardware.xacro (robot description, xacro)
@@ -1,13 +1,13 @@
 <?xml version="1.0"?>
-<robot>
-  <property name="M_PI" value="3.14159"/>
-  <property name="M_SCALE" value="0.01"/>
-  <property name="HOKUYO_RADIUS" value="0.02"/>
-  <property name="HOKUYO_LENGTH" value="0.07"/>
-  <property name="KINECT_LENGTH" value="0.064"/>
-  <property name="KINECT_WIDTH" value="0.121"/>
-  <property name="KINECT_HEIGHT" value="0.0381"/>
+<robot xmlns:xacro="http://www.ros.org/wiki/xacro">
+  <xacro:property name="M_PI" value="3.14159"/>
+  <xacro:property name="M_SCALE" value="0.01"/>
+  <xacro:property name="HOKUYO_RADIUS" value="0.02"/>
+  <xacro:property name="HOKUYO_LENGTH" value="0.07"/>
+  <xacro:property name="KINECT_LENGTH" value="0.064"/>
+  <xacro:property name="KINECT_WIDTH" value="0.121"/>
+  <xacro:property name="KINECT_HEIGHT" value="0.0381"/>
   <!-- WHEEL -->
-  <macro name="wheel" params="parent name *origin *axis">
+  <xacro:macro name="wheel" params="parent name *origin *axis">
     <joint name="${name}_joint" type="continuous">
       <insert_block name="origin" />
@@ -31,7 +31,7 @@
       </visual>
     </link>
-  </macro>
+  </xacro:macro>
   <!-- COMMAND BRIDGE -->
-  <macro name="command_bridge" params="parent name *origin">
+  <xacro:macro name="command_bridge" params="parent name *origin">
     <joint name="${name}_joint" type="fixed">
       <insert_block name="origin" />
@@ -54,7 +54,7 @@
       </collision>
     </link>
-  </macro>
+  </xacro:macro>
   <!-- LASER SCANNER -->
-  <macro name="laser" params="parent name *origin">
+  <xacro:macro name="laser" params="parent name *origin">
     <joint name="${name}_joint" type="fixed">
       <insert_block name="origin" />
@@ -83,7 +83,7 @@
       </collision>
     </link>
-  </macro>
+  </xacro:macro>
   <!-- Camera -->
-  <macro name="camera" params="parent name *origin">
+  <xacro:macro name="camera" params="parent name *origin">
     <joint name="${name}_joint" type="fixed">
       <insert_block name="origin" />
@@ -106,7 +106,7 @@
       </visual>
     </link>
-  </macro>
+  </xacro:macro>
   <!-- AngleBracket With USB Hub -->
-  <macro name="anglebracketusb" params="parent name *origin">
+  <xacro:macro name="anglebracketusb" params="parent name *origin">
     <joint name="${name}_joint" type="fixed">
       <insert_block name="origin" />
@@ -129,7 +129,7 @@
       </visual>
     </link>
-  </macro>
+  </xacro:macro>
   <!-- KINECT -->
-  <macro name="kinect" params="parent name color llimit ulimit vlimit *origin">
+  <xacro:macro name="kinect" params="parent name color llimit ulimit vlimit *origin">
     <joint name="${name}_joint" type="revolute">
       <insert_block name="origin" />
@@ -161,4 +161,4 @@
       </collision>
     </link>
-  </macro>
+  </xacro:macro>
 </robot>
